File: Eagle/BrewDoo.brd (EAGLE design)
At the start: 25 parts, among them IC1 ATMEGA328P, Q1 16MHz

Commit message: Version 1.0.
Parts:
- added H5, H6, H7, H8: MOUNT-HOLE3.0, holes:3,0
- moved R2 7.41 mm to (85.1, 8.89)
- moved X1 6.48 mm to (20.3, 5.08)
- moved R4 6.35 mm to (80.0, 21.6), turned to 45 degrees
- moved R3 4.58 mm to (76.2, 7.62)
- moved LED_A 0.64 mm to (97.2, 34.3)
- moved LED_B 0.64 mm to (97.2, 20.3)
Routing:
- net N$6: track 3.17 -> 14.0 mm
- net N$16: track 17.6 -> 27.9 mm
- net N$4: track 73.5 -> 66.9 mm
- net N$17: track 23.5 -> 19.4 mm
- net N$11: track 131.5 -> 128.5 mm
- net N$20: track 31.1 -> 34.0 mm
- net N$18: track 33.1 -> 30.4 mm
- net +5V: track 164.6 -> 165.9 mm
- net N$21: track 10.1 -> 10.7 mm
Changed lines of the file:
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@@
 <element name="H3" library="holes" package="5,0" value="MOUNT-HOLE5.0" x="101.6" y="0"/>
 <element name="H4" library="holes" package="5,0" value="MOUNT-HOLE5.0" x="101.6" y="50.8"/>
-<element name="R2" library="rcl" package="0207/12" value="270" x="91.44" y="12.7" rot="R90"/>
-<element name="R3" library="rcl" package="0207/10" value="270" x="80.01" y="10.16"/>
-<element name="R4" library="rcl" package="0207/10" value="270" x="80.01" y="15.24"/>
+<element name="R2" library="rcl" package="0207/12" value="270" x="85.09" y="8.89" rot="R90"/>
+<element name="R3" library="rcl" package="0207/10" value="270" x="76.2" y="7.62"/>
+<element name="R4" library="rcl" package="0207/10" value="270" x="80.01" y="21.59" rot="R45"/>
 <element name="R5" library="rcl" package="0207/15" value="270" x="77.47" y="31.75"/>
 <element name="R6" library="rcl" package="0207/15" value="270" x="74.93" y="29.21"/>
 <element name="R7" library="rcl" package="0207/15" value="270" x="76.2" y="36.83"/>
-<element name="LED_A" library="LEDs-pk" package="RGBLED_STAGG" value="RGBLED_CC_STAG" x="96.52" y="34.29"/>
-<element name="LED_B" library="LEDs-pk" package="RGBLED_STAGG" value="RGBLED_CC_STAG" x="96.52" y="20.32"/>
-<element name="X1" library="con-ptr500" package="AK300/2" value="" x="13.97" y="6.35" rot="R270">
-<attribute name="OC_NEWARK" value="unknown" x="13.97" y="6.35" size="1.778" layer="27" rot="R270" display="off"/>
-<attribute name="MPN" value="" x="13.97" y="6.35" size="1.778" layer="27" rot="R270" display="off"/>
-<attribute name="MF" value="" x="13.97" y="6.35" size="1.778" layer="27" rot="R270" display="off"/>
-<attribute name="OC_FARNELL" value="unknown" x="13.97" y="6.35" size="1.778" layer="27" rot="R270" display="off"/>
+<element name="LED_A" library="LEDs-pk" package="RGBLED_STAGG" value="RGBLED_CC_STAG" x="97.155" y="34.29"/>
+<element name="LED_B" library="LEDs-pk" package="RGBLED_STAGG" value="RGBLED_CC_STAG" x="97.155" y="20.32"/>
+<element name="X1" library="con-ptr500" package="AK300/2" value="" x="20.32" y="5.08" rot="R270">
+<attribute name="OC_NEWARK" value="unknown" x="20.32" y="5.08" size="1.778" layer="27" rot="R270" display="off"/>
+<attribute name="MPN" value="" x="20.32" y="5.08" size="1.778" layer="27" rot="R270" display="off"/>
+<attribute name="MF" value="" x="20.32" y="5.08" size="1.778" layer="27" rot="R270" display="off"/>
+<attribute name="OC_FARNELL" value="unknown" x="20.32" y="5.08" size="1.778" layer="27" rot="R270" display="off"/>
 </element>
 <element name="U$1" library="jumper-wires-pk" package="WIRE-0.3" value="WIRE-0.3" x="31.75" y="15.24" rot="R180"/>
 <element name="U$2" library="jumper-wires-pk" package="WIRE-0.3" value="WIRE-0.3" x="31.75" y="11.43"/>
 <element name="U$3" library="jumper-wires-pk" package="WIRE-0.6" value="WIRE-0.6" x="13.97" y="20.32" rot="R90"/>
+<element name="H5" library="holes" package="3,0" value="MOUNT-HOLE3.0" x="15.875" y="44.45"/>
+<element name="H6" library="holes" package="3,0" value="MOUNT-HOLE3.0" x="91.44" y="44.45"/>
+<element name="H7" library="holes" package="3,0" value="MOUNT-HOLE3.0" x="91.44" y="12.7"/>
+<element name="H8" library="holes" package="3,0" value="MOUNT-HOLE3.0" x="8.89" y="8.89"/>
 </elements>
 <signals>
@@
 <contactref element="X1" pad="1"/>
 <wire x1="15.924015625" y1="27.74005625" x2="16" y2="28" width="0.8128" layer="16"/>
-<wire x1="13.97" y1="8.8646" x2="13.97" y2="12.7" width="0.8128" layer="16"/>
-<wire x1="13.97" y1="12.7" x2="25.4" y2="12.7" width="0.8128" layer="16"/>
 <wire x1="25.4" y1="12.7" x2="27.94" y2="15.24" width="0.8128" layer="16"/>
 <wire x1="27.94" y1="15.24" x2="35.56" y2="15.24" width="0.8128" layer="1"/>
@@
 <wire x1="26.67" y1="48.26" x2="24.13" y2="46.99" width="0.8128" layer="16"/>
 <wire x1="24.13" y1="46.99" x2="24.13" y2="44.45" width="0.8128" layer="16"/>
+<wire x1="20.32" y1="7.5946" x2="20.32" y2="12.7" width="0.8128" layer="16"/>
+<wire x1="20.32" y1="12.7" x2="25.4" y2="12.7" width="0.8128" layer="16"/>
+<wire x1="13.97" y1="12.7" x2="20.32" y2="12.7" width="0.8128" layer="16"/>
 </signal>
 <signal name="N$5">
@@
 <wire x1="67.31" y1="48.26" x2="74.93" y2="48.26" width="0.8128" layer="16"/>
 <wire x1="74.93" y1="48.26" x2="80.01" y2="43.18" width="0.8128" layer="16"/>
-<wire x1="80.01" y1="43.18" x2="80.01" y2="5.08" width="0.8128" layer="16"/>
-<wire x1="80.01" y1="5.08" x2="35.56" y2="5.08" width="0.8128" layer="16"/>
 <wire x1="35.56" y1="5.08" x2="33.02" y2="7.62" width="0.8128" layer="16"/>
 <wire x1="33.02" y1="7.62" x2="33.02" y2="17.78" width="0.8128" layer="16"/>
@@
 <wire x1="60.96" y1="41.91" x2="52.07" y2="41.91" width="0.8128" layer="16"/>
 <wire x1="52.07" y1="41.91" x2="52.07" y2="44.45" width="0.8128" layer="16"/>
+<wire x1="35.56" y1="5.08" x2="74.93" y2="5.08" width="0.8128" layer="16"/>
+<wire x1="74.93" y1="5.08" x2="80.01" y2="10.16" width="0.8128" layer="16"/>
+<wire x1="80.01" y1="10.16" x2="80.01" y2="43.18" width="0.8128" layer="16"/>
 </signal>
 <signal name="N$12">
@@
 <contactref element="R2" pad="2"/>
 <contactref element="LED_B" pad="RED"/>
-<wire x1="91.44" y1="19.05" x2="94.615" y2="19.05" width="0.8128" layer="16"/>
+<wire x1="85.09" y1="15.24" x2="85.09" y2="19.05" width="0.8128" layer="16"/>
+<wire x1="85.09" y1="19.05" x2="95.25" y2="19.05" width="0.8128" layer="16"/>
 </signal>
 <signal name="N$16">
 <contactref element="R3" pad="2"/>
 <contactref element="LED_B" pad="GREEN"/>
-<wire x1="85.09" y1="10.16" x2="92.71" y2="10.16" width="0.8128" layer="16"/>
-<wire x1="92.71" y1="10.16" x2="97.155" y2="19.05" width="0.8128" layer="16"/>
+<wire x1="81.28" y1="7.62" x2="97.79" y2="7.62" width="0.8128" layer="16"/>
+<wire x1="97.79" y1="7.62" x2="97.79" y2="19.05" width="0.8128" layer="16"/>
 </signal>
 <signal name="N$17">
 <contactref element="R4" pad="2"/>
 <contactref element="LED_B" pad="BLUE"/>
-<wire x1="85.09" y1="15.24" x2="85.09" y2="24.13" width="0.8128" layer="16"/>
-<wire x1="85.09" y1="24.13" x2="96.52" y2="24.13" width="0.8128" layer="16"/>
-<wire x1="96.52" y1="24.13" x2="98.425" y2="21.59" width="0.8128" layer="16"/>
+<wire x1="83.6021" y1="25.1821" x2="83.82" y2="25.4" width="0.8128" layer="16"/>
+<wire x1="83.82" y1="25.4" x2="99.06" y2="25.4" width="0.8128" layer="16"/>
+<wire x1="99.06" y1="25.4" x2="99.06" y2="21.59" width="0.8128" layer="16"/>
 </signal>
 <signal name="N$13">
@@
 <contactref element="LED_A" pad="RED"/>
 <wire x1="85.09" y1="31.75" x2="86.36" y2="33.02" width="0.8128" layer="16"/>
-<wire x1="86.36" y1="33.02" x2="94.615" y2="33.02" width="0.8128" layer="16"/>
+<wire x1="86.36" y1="33.02" x2="95.25" y2="33.02" width="0.8128" layer="16"/>
 </signal>
 <signal name="N$22">
@@
 <contactref element="LED_A" pad="GREEN"/>
 <wire x1="82.55" y1="29.21" x2="95.25" y2="29.21" width="0.8128" layer="16"/>
-<wire x1="95.25" y1="29.21" x2="97.155" y2="33.02" width="0.8128" layer="16"/>
+<wire x1="95.25" y1="29.21" x2="97.79" y2="33.02" width="0.8128" layer="16"/>
 </signal>
 <signal name="N$23">
 <contactref element="R7" pad="2"/>
 <contactref element="LED_A" pad="BLUE"/>
-<wire x1="98.425" y1="35.56" x2="96.52" y2="39.37" width="0.8128" layer="16"/>
+<wire x1="99.06" y1="35.56" x2="96.52" y2="39.37" width="0.8128" layer="16"/>
 <wire x1="96.52" y1="39.37" x2="86.36" y2="39.37" width="0.8128" layer="16"/>
 <wire x1="86.36" y1="39.37" x2="83.82" y2="36.83" width="0.8128" layer="16"/>
@@
 <contactref element="IC1" pad="5"/>
 <contactref element="R2" pad="1"/>
-<wire x1="34.29" y1="3.81" x2="30.48" y2="7.62" width="0.8128" layer="16"/>
 <wire x1="30.48" y1="7.62" x2="30.48" y2="17.78" width="0.8128" layer="16"/>
-<wire x1="34.29" y1="3.81" x2="87.63" y2="3.81" width="0.8128" layer="16"/>
-<wire x1="87.63" y1="3.81" x2="91.44" y2="6.35" width="0.8128" layer="16"/>
+<wire x1="30.48" y1="7.62" x2="35.56" y2="2.54" width="0.8128" layer="16"/>
+<wire x1="35.56" y1="2.54" x2="85.09" y2="2.54" width="0.8128" layer="16"/>
 </signal>
 <signal name="N$18">
@@
 <contactref element="R3" pad="1"/>
 <wire x1="45.72" y1="17.78" x2="45.72" y2="16.51" width="0.8128" layer="16"/>
-<wire x1="45.72" y1="16.51" x2="52.07" y2="10.16" width="0.8128" layer="16"/>
-<wire x1="52.07" y1="10.16" x2="74.93" y2="10.16" width="0.8128" layer="16"/>
+<wire x1="45.72" y1="16.51" x2="54.61" y2="7.62" width="0.8128" layer="16"/>
+<wire x1="54.61" y1="7.62" x2="71.12" y2="7.62" width="0.8128" layer="16"/>
 </signal>
 <signal name="N$20">
@@
 <wire x1="70.54" y1="12" x2="52.8" y2="12" width="0.8" layer="16"/>
 <wire x1="48" y1="17.6" x2="48.26" y2="17.78" width="0.8" layer="16"/>
-<wire x1="70.54" y1="12" x2="74.93" y2="15.24" width="0.8" layer="16"/>
+<wire x1="70.54" y1="12" x2="76.417896875" y2="17.997896875" width="0.8" layer="16"/>
 </signal>
 <signal name="RESET">
